File: MainPCB/revision 1.2d/DCHDMI.sch (KiCad schematic (older format))
At the start: 81 parts, among them CON1 3-1775333-2, CON2 2001-1-2-21-00-BK, CON3 CONN_01X06, CON4 CONN_01X03, U1 MCP1826S-1202E/DB, U2 MIC5219-2.5YM5-TR, U3 LP5907MFX-1.8/NOPB, U4 ADV7513, U5 664G-03LF, U6 10CL025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

Commit message: Added 1.2d
Parts:
- added C41, C46, C47: 47p, Capacitors_SMD:C_0603_HandSoldering, symbol C_Small
- added C48: .1u, Capacitors_SMD:C_0603_HandSoldering, symbol C_Small
- added C49: 22u, Capacitors_SMD:C_0603_HandSoldering, symbol C_Small
- added R18, R19, R20, R7: 10K, Capacitors_SMD:C_0603_HandSoldering, symbol R_Small
Connections:
- net +3V3: now also C48.1, C49.1, R18.2, R19.2, R7.1; no longer U6.9 (nSTATUS)
- net ABCK: now also C46.2
- net ADAT: now also C47.2
- net ALRK: now also C41.2
- net GND: now also U6.145 (THERMAL), C41.1, C46.1, C47.1, C48.2, C49.2, R20.2; no longer U6.21 (nCE)
- net TDI: now also R19.1
- net TMS: now also R18.1
- net nCE: now reaches U8.13 (IO4)
- net nCE: now also U6.21 (nCE), R20.1
- new net: R7.2, U6.9 (nSTATUS)
- no-connect marks 26 -> 25
