File: MainPCB/revision 1.2d/DCHDMI.kicad_pcb (KiCad board)
At the start: 4 copper layers, 66.6 x 51.3 mm, 108 parts, among them CON1 3-1775333-2, CON2 2001-1-2-21-00-BK, U1 MCP1826S-1202E/DB, U2 MIC5219-2.5YM5-TR, U3 LP5907MFX-1.8/NOPB, U4 ADV7513, U5 664G-03LF, U6 10CL025, U7 MX25L1606EM1I-12G, U8 ESP-12E

Commit message: Increased version number
Other:
- board text added: "DCHDMI 1.2e"
- board text removed: "DCHDMI 1.2d"
Changed lines of the file:
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@@
     (links 432)
     (no_connects 2)
-    (area 121.924999 73.596999 188.643001 125.075001)
+    (area 121.924999 72.324999 188.643001 125.075001)
     (thickness 1.6)
     (drawings 58)
@@
     (effects (font (size 1 1) (thickness 0.1)))
   )
-  (gr_text "DCHDMI 1.2d" (at 170.45 101.85) (layer F.SilkS)
+  (gr_text "DCHDMI 1.2e" (at 170.45 101.85) (layer F.SilkS)
     (effects (font (size 1.5 1.5) (thickness 0.25)))
   )
