File: MainPCB/revision 1.2e/DCHDMI.sch (KiCad schematic (older format))
At the start: 90 parts, among them CON1 3-1775333-2, CON2 2001-1-2-21-00-BK, CON3 CONN_01X06, CON4 CONN_01X03, U1 MCP1826S-1202E/DB, U2 MIC5219-2.5YM5-TR, U3 LP5907MFX-1.8/NOPB, U4 ADV7513, U5 664G-03LF, U6 10CL025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

Commit message: Minor Update to Edge Cuts
Parts:
- C49: footprint Capacitors_SMD:C_0603_HandSoldering -> Capacitors_SMD:C_0805_HandSoldering
Changed lines of the file:
@@
 F 0 "C49" H 8160 10420 50  0000 L CNN
 F 1 "22u" H 8160 10270 50  0000 L CNN
-F 2 "Capacitors_SMD:C_0603_HandSoldering" H 8150 10350 50  0001 C CNN
+F 2 "Capacitors_SMD:C_0805_HandSoldering" H 8150 10350 50  0001 C CNN
 F 3 "" H 8150 10350 50  0000 C CNN
 	1    8150 10350
