File: MainPCB/revision 1.2f/DCHDMI.sch (KiCad schematic (older format))
At the start: 90 parts, among them CON1 3-1775333-2, CON2 2001-1-2-21-00-BK, CON3 CONN_01X06, CON4 CONN_01X03, U1 MCP1826S-1202E/DB, U2 MIC5219-2.5YM5-TR, U3 LP5907MFX-1.8/NOPB, U4 ADV7513, U5 664G-03LF, U6 10CL025, U7 MX25L1606EM1I-12G, U8 ESP-12E

Commit message: 1.2 Revison
JTAG replaced with ESP header.  In Game Reset Pads added.
Parts:
- removed C50: .1u, Capacitors_SMD:C_0603_HandSoldering, symbol C_Small
- removed D5, D6: B5819WS, Diodes_SMD:D_SOD-323_HandSoldering, symbol D_Schottky_Small
- removed R1, R18: 10K, Capacitors_SMD:C_0603_HandSoldering, symbol R_Small
- added CON5: CONN_01X03, pads:2_Pads_Small, symbol DCHDMI-rescue:CONN_01X03
- added SW1: SW_DIP_x02, Buttons_Switches_SMD:SW_DIP_x2_W7.62mm_Slide_Copal_CHS-B, symbol Switch:SW_DIP_x02
- C1, C10, C11, C12, C13, C14, C15, C16, C17, C18, C19, C2, C20, C21, C22, C23, C24, C25, C26, C27, C28, C29, C3, C30, C31, C32, C33, C34, C35, C36, C37, C38, C39, C4, C40, C41, C42, C43, C44, C45, C46, C47, C48, C49, C5, C6, C7, C8, C9: symbol C_Small -> Device:C_Small
- CON1: symbol 3-1775333-2 -> dk_Rectangular-Connectors-Headers-Male-Pins:3-1775333-2
- CON2: value 2001-1-2-21-00-BK -> DC2R019JA7R1700; footprint digikey-footprints:HDMI_Mini_Female_2001-1-2-21-00-BK -> jumper:DC2R019JA7R1700; symbol 2001-1-2-21-00-BK -> dk_USB-DVI-HDMI-Connectors:2001-1-2-21-00-BK
- CON3: symbol CONN_01X06 -> DCHDMI-rescue:CONN_01X06
- CON4: symbol CONN_01X03 -> DCHDMI-rescue:CONN_01X03
- D1: symbol Led_Small -> DCHDMI-rescue:Led_Small
- D2, D3, D4: symbol SP3012-04UTG -> dk_TVS-Diodes:SP3012-04UTG
- L1, L2, L3: symbol L_Small -> Device:L_Small
- R10, R11, R12, R13, R14, R15, R16, R17, R2, R20, R3, R4, R5, R6, R7, R8, R9: symbol R_Small -> Device:R_Small
- U1: symbol MCP1826S-1202E/DB -> DCHDMI-rescue:MCP1826S-1202E_DB
- U2: symbol MIC5219-2.5YM5-TR -> dk_PMIC-Voltage-Regulators-Linear:MIC5219-2.5YM5-TR
- U3: symbol LP5907MFX-1.8/NOPB -> DCHDMI-rescue:LP5907MFX-1.8_NOPB
- U4: symbol ADV7513 -> DCHDMI-rescue:ADV7513
- U5: symbol 664G-03LF -> dk_Clock-Timing-Clock-Generators-PLLs-Frequency-Synthesizers:664G-03LF
- U6: symbol 10CL025 -> DCHDMI-rescue:10CL025
- U7: symbol MX25L1606EM1I-12G -> dk_Memory:MX25L1606EM1I-12G
- U8: symbol ESP-12E -> ESP12:ESP-12E
Connections:
- net labels added: HRST, HRST_OUT, RXD, SRST, TXD
- net labels removed: RX, TX
- wire segments 476 -> 655
- no-connect marks 29 -> 30
Other:
- moved on the sheet: CON4
