File: MainPCB/revision 1.3/DCHDMI.sch (KiCad schematic (older format))
At the start: 87 parts, among them CON1 3-1775333-2, CON2 DC2R019JA7R1700, CON3 CONN_01X06, CON4 CONN_01X03, CON5 CONN_01X03, SW1 SW_DIP_x02, U1 MCP1826S-1202E/DB, U2 MIC5219-2.5YM5-TR, U3 LP5907MFX-1.8/NOPB, U4 ADV7513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

Commit message: Added 470 series resistor
Parts:
- added R1: 470, Capacitors_SMD:C_0603_HandSoldering, symbol Device:R_Small
Connections:
- wire segments 655 -> 657
Changed lines of the file:
@@
 Text Label 10500 9650 2    51   ~ 0
 HRST
-Text Label 11100 9650 0    51   ~ 0
+Text Label 11700 9650 0    51   ~ 0
 HRST_OUT
 Text Label 8850 7650 0    51   ~ 0
@@
 	2950 8600 2950 8800
 NoConn ~ 8400 9500
+$Comp
+L Device:R_Small R1
+U 1 1 5B96ECCA
+P 11450 9650
+F 0 "R1" V 11400 9600 50  0000 L BNN
+F 1 "470" V 11550 9600 50  0000 L BNN
+F 2 "Capacitors_SMD:C_0603_HandSoldering" H 11450 9650 50  0001 C CNN
+F 3 "" H 11450 9650 50  0000 C CNN
+	1    11450 9650
+	0    1    1    0
+$EndComp
+Wire Wire Line
+	11100 9650 11350 9650
+Wire Wire Line
+	11550 9650 11700 9650
 $EndSCHEMATC

Commit message: Fixed Issue
Parts:
- added R18: 470, Capacitors_SMD:C_0603_HandSoldering, symbol Device:R_Small
Connections:
- wire segments 657 -> 660
Changed lines of the file:
@@
 Text Label 8850 7750 0    51   ~ 0
 SRST
-Text Label 2850 2100 2    51   ~ 0
+Text Label 2950 2300 0    51   ~ 0
 SRST
 Wire Wire Line
-	2850 2100 2850 1950
+	2750 2050 2850 1950
 Wire Wire Line
 	2850 1950 2950 1950
@@
 Wire Wire Line
 	11550 9650 11700 9650
+$Comp
+L Device:R_Small R18
+U 1 1 5B986708
+P 2750 2150
+F 0 "R18" V 2700 2100 50  0000 L BNN
+F 1 "470" V 2850 2100 50  0000 L BNN
+F 2 "Capacitors_SMD:C_0603_HandSoldering" H 2750 2150 50  0001 C CNN
+F 3 "" H 2750 2150 50  0000 C CNN
+	1    2750 2150
+	-1   0    0    1
+$EndComp
+Wire Wire Line
+	2750 2250 2900 2250
+Wire Wire Line
+	2900 2250 2900 2300
+Wire Wire Line
+	2900 2300 2950 2300
 $EndSCHEMATC
